File: connectors.kicad_sch (KiCad schematic)
At the start: 27 parts, among them J1 2001-1-2-21-00-BK, J2 JC-128, P2 HOST, P3 CAM1, P4 CONN_02X20, Q3 2N7002P.215

Commit message: fix missing hdmi junctions, dangling trace
Connections:
- net HDMI_SCL: now also D5.3 (common), R4.2
- net HDMI_SDA: now also D6.3 (common), R5.2
Changed lines of the file:
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@@
+	)
+	(junction
+		(at 218.44 64.77)
+		(diameter 0)
+		(color 0 0 0 0)
 	)
 	(junction
@@
 	(junction
 		(at 102.87 69.85)
+		(diameter 0)
+		(color 0 0 0 0)
+	)
+	(junction
+		(at 231.14 67.31)
 		(diameter 0)
 		(color 0 0 0 0)
@@
 	(wire
 		(pts
+			(xy 231.14 67.31) (xy 234.95 67.31)
+		)
+		(stroke
+			(width 0)
+			(type default)
+		)
+	)
+	(wire
+		(pts
 			(xy 104.14 17.78) (xy 104.14 41.91)
 		)
@@
 	(wire
 		(pts
-			(xy 173.99 67.31) (xy 234.95 67.31)
+			(xy 173.99 67.31) (xy 231.14 67.31)
 		)
 		(stroke
@@
 	(wire
 		(pts
-			(xy 218.44 43.18) (xy 218.44 87.63)
+			(xy 218.44 43.18) (xy 218.44 64.77)
+		)
+		(stroke
+			(width 0)
+			(type default)
+		)
+	)
+	(wire
+		(pts
+			(xy 231.14 67.31) (xy 231.14 87.63)
 		)
 		(stroke
@@
 	(wire
 		(pts
-			(xy 231.14 43.18) (xy 231.14 87.63)
+			(xy 231.14 43.18) (xy 231.14 67.31)
 		)
 		(stroke
@@
 	(wire
 		(pts
+			(xy 218.44 64.77) (xy 218.44 87.63)
+		)
+		(stroke
+			(width 0)
+			(type default)
+		)
+	)
+	(wire
+		(pts
 			(xy 58.42 24.13) (xy 60.96 24.13)
 		)
@@
 	(wire
 		(pts
-			(xy 173.99 64.77) (xy 234.95 64.77)
+			(xy 173.99 64.77) (xy 218.44 64.77)
 		)
 		(stroke
@@
 		)
 		(stroke
+			(width 0)
+			(type default)
+		)
+	)
+	(wire
+		(pts
+			(xy 218.44 64.77) (xy 234.95 64.77)
+		)
+		(stroke
